File: electronics/substrate_adapter/substrate_adapter.kicad_pcb (KiCad board)
At the start: 2 copper layers, 25.4 x 25.4 mm, 18 parts, among them J1 PIX1, J10 R_CONN, J11 PIX1, J12 PIX2, J13 PIX3, J14 BOT_TCE, J15 TOP_TCE, J16 PIX4, J17 PIX5, J18 PIX6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

Commit message: update silk
Other:
- board text added: "45f1e60"
Changed lines of the file:
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@@
   (general
     (thickness 1.6)
-    (drawings 8)
+    (drawings 10)
     (tracks 57)
     (zones 0)
@@
   )
   (setup
-    (last_trace_width 1)
+    (last_trace_width 0.25)
     (user_trace_width 1)
     (trace_clearance 0.2)
@@
     )
   )
+  (gr_text 45f1e60 (at -7 12) (layer B.SilkS)
+    (effects (font (size 1 1) (thickness 0.15)) (justify mirror))
+  )
+  (gr_text 45f1e60 (at -7 12) (layer F.SilkS)
+    (effects (font (size 1 1) (thickness 0.15)))
+  )
   (gr_line (start 8 8) (end -8 8) (layer Edge.Cuts) (width 0.05))
